File: hardware/BREAD_Slice.kicad_pcb (KiCad board)
At the start: 2 copper layers, 70 x 100 mm, 22 parts, among them J1 Conn_01x10_Socket, SW1 SW_DIP_x04, U1 AP63205

Commit message: Finished draft 1, still need documentation and review
Parts:
- added D3: MM3Z18VT1G, Diode_SMD:D_SOD-323, F.Cu at (177.0, 122.0)
- added J2: Screw_Terminal_01x06, TerminalBlock_Phoenix:TerminalBlock_Phoenix_PT-1,5-6-3.5-H_1x06_P3.50mm_Horizontal, F.Cu at (183.8, 72.8)
- added J3: Screw_Terminal_01x02, TerminalBlock_Phoenix:TerminalBlock_Phoenix_PT-1,5-2-3.5-H_1x02_P3.50mm_Horizontal, F.Cu at (183.5, 118.8)
- added J4: Screw_Terminal_01x08, TerminalBlock_Phoenix:TerminalBlock_Phoenix_PT-1,5-8-3.5-H_1x08_P3.50mm_Horizontal, F.Cu at (183.8, 103.2)
- added R1: 1k, Resistor_SMD:R_0603_1608Metric, F.Cu at (142.3, 67.8)
- added R10: 1k, Resistor_SMD:R_0603_1608Metric, F.Cu at (177.0, 62.2)
- added R11: 1k, Resistor_SMD:R_0603_1608Metric, F.Cu at (177.1, 58.8)
- added R12: 1k, Resistor_SMD:R_0603_1608Metric, F.Cu at (177.0, 55.2)
- added R13: 2.4k, Resistor_SMD:R_0603_1608Metric, F.Cu at (167.8, 103.1)
- added R14: 2.4k, Resistor_SMD:R_0603_1608Metric, F.Cu at (167.8, 96.0)
- added R15: 2.4k, Resistor_SMD:R_0603_1608Metric, F.Cu at (167.8, 89.1)
- added R16: 47, Resistor_SMD:R_0603_1608Metric, F.Cu at (177.8, 103.0)
- added R17: 47, Resistor_SMD:R_0603_1608Metric, F.Cu at (177.8, 96.0)
- added R18: 47, Resistor_SMD:R_0603_1608Metric, F.Cu at (177.8, 89.0)
- added R19: 2.4k, Resistor_SMD:R_0603_1608Metric, F.Cu at (167.8, 82.0)
- added R2: 1k, Resistor_SMD:R_0603_1608Metric, F.Cu at (159.2, 68.0)
- added R20: 47, Resistor_SMD:R_0603_1608Metric, F.Cu at (177.8, 82.0)
- added R21: 100k, Resistor_SMD:R_0603_1608Metric, F.Cu at (172.8, 120.5)
- added R3: 1k, Resistor_SMD:R_0603_1608Metric, F.Cu at (142.2, 61.0)
- added R4: 1k, Resistor_SMD:R_0603_1608Metric, F.Cu at (159.2, 60.6)
- added R5: 1k, Resistor_SMD:R_0603_1608Metric, F.Cu at (142.2, 54.0)
- added R6: 1k, Resistor_SMD:R_0603_1608Metric, F.Cu at (159.2, 54.0)
- added R7: 1k, Resistor_SMD:R_0603_1608Metric, F.Cu at (177.0, 72.8)
- added R8: 1k, Resistor_SMD:R_0603_1608Metric, F.Cu at (177.0, 69.0)
- added R9: 1k, Resistor_SMD:R_0603_1608Metric, F.Cu at (177.0, 65.8)
- added SW3: SW_SPDT, Button_Switch_THT:SW_Slide-03_Wuerth-WS-SLTV_10x2.5x6.4_P2.54mm, F.Cu at (167.8, 117.0)
- added U10: CPC1002N, Package_SO:SOP-4_3.8x4.1mm_P2.54mm, F.Cu at (172.8, 87.0)
- added U11: CPC1002N, Package_SO:SOP-4_3.8x4.1mm_P2.54mm, F.Cu at (172.8, 80.0)
- added U12: NTGS4111PT1G, Package_TO_SOT_SMD:TSOT-23-6, F.Cu at (176.9, 118.8)
- added U2: LTV-817S, Package_DIP:SMDIP-4_W9.53mm, F.Cu at (150.5, 68.0)
- added U3: LTV-817S, Package_DIP:SMDIP-4_W9.53mm, F.Cu at (167.5, 68.0)
- added U4: LTV-817S, Package_DIP:SMDIP-4_W9.53mm, F.Cu at (150.5, 61.0)
- added U5: LTV-817S, Package_DIP:SMDIP-4_W9.53mm, F.Cu at (167.5, 61.0)
- added U6: LTV-817S, Package_DIP:SMDIP-4_W9.53mm, F.Cu at (150.5, 54.0)
- added U7: LTV-817S, Package_DIP:SMDIP-4_W9.53mm, F.Cu at (167.5, 54.0)
- added U8: CPC1002N, Package_SO:SOP-4_3.8x4.1mm_P2.54mm, F.Cu at (172.8, 101.0)
- added U9: CPC1002N, Package_SO:SOP-4_3.8x4.1mm_P2.54mm, F.Cu at (172.8, 94.0)
Connections:
- A1 pad 10: /slice_template/D7 -> /IN3
- A1 pad 11: /slice_template/D8 -> /IN5
- A1 pad 12: /slice_template/D9 -> /IN6
- A1 pad 13: /slice_template/D10 -> /IN4
- A1 pad 14: /slice_template/D11/MOSI -> /IN2
- A1 pad 19: /slice_template/A0 -> OUT1
- A1 pad 20: /slice_template/A1 -> OUT2
- A1 pad 21: /slice_template/A2 -> OUT3
- A1 pad 22: /slice_template/A3 -> OUT4
- A1 pad 9: /slice_template/D6 -> /IN1
Routing:
- net +5V: track 104.2 -> 194.6 mm, vias 1 -> 7
- net /IN6: track 0.00 -> 83.4 mm, vias 0 -> 1
- net /IN5: track 0.00 -> 81.6 mm, vias 0 -> 1
- net /IN4: track 0.00 -> 79.3 mm, vias 0 -> 1
- net /IN2: track 0.00 -> 74.5 mm, vias 0 -> 1
- net +12V: track 52.1 -> 124.1 mm
- net /IN3: track 0.00 -> 70.8 mm, vias 0 -> 1
- net VOUT: track 0.00 -> 69.5 mm
- net /IN1: track 0.00 -> 60.6 mm, vias 0 -> 1
- net OUT4: track 0.00 -> 46.2 mm
- net OUT3: track 0.00 -> 41.6 mm
- net OUT2: track 0.00 -> 36.9 mm
- net OUT1: track 0.00 -> 32.7 mm
- net Net-(R11-Pad1): track 0.00 -> 22.4 mm
- net Net-(R9-Pad1): track 0.00 -> 22.4 mm
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- added copper zone on F.Cu, net /24V
- added copper zone on F.Cu, net GND
Other:
- board text added: "+"
- board text added: "-"
- board text added: "I1"
- board text added: "I2"
- board text added: "I3"
- board text added: "I4"
- board text added: "I5"
- board text added: "I6"
- board text added: "O1+"
- board text added: "O1-"
- board text added: "O2+"
- board text added: "O2-"
- board text added: "O3+"
- board text added: "O3-"
- board text added: "O4+"
- board text added: "O4-"

Commit message: some revisions and schem and brd
Parts:
- moved U2 20.1 mm to (164.9, 82.0)
- moved R1 19.0 mm to (156.7, 80.1), turned to 90 degrees
- moved U4 15.8 mm to (164.8, 67.7)
- moved R3 15.2 mm to (156.6, 66.0), turned to 90 degrees
- moved R5 14.7 mm to (156.7, 51.3), turned to 90 degrees
- moved U6 14.5 mm to (164.9, 53.0)
- moved R7 11.2 mm to (173.2, 83.2)
- moved R6 10.2 mm to (156.6, 44.2), turned to 90 degrees
- moved U10 9.85 mm to (172.8, 96.9)
- moved U8 9.85 mm to (172.8, 110.9)
- moved U9 9.85 mm to (172.8, 103.9)
- moved J4 9.85 mm to (183.8, 113.1)
- moved R13 9.85 mm to (167.8, 112.9)
- moved R14 9.85 mm to (167.8, 105.8)
- moved R15 9.85 mm to (167.8, 98.9)
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Routing:
- net +5V: track 194.6 -> 96.5 mm, vias 7 -> 1
- net /IN6: track 83.4 -> 4.94 mm
- net /IN5: track 81.6 -> 5.19 mm
- net /IN4: track 79.3 -> 4.73 mm
- net /IN2: track 74.5 -> 4.95 mm
- net /IN3: track 70.8 -> 4.95 mm
- net /IN1: track 60.6 -> 4.84 mm
- net Net-(R11-Pad1): track 22.4 -> 0.00 mm
- net Net-(R9-Pad1): track 22.4 -> 0.00 mm
- net Net-(R7-Pad1): track 22.3 -> 0.00 mm
- net OUT1: track 32.7 -> 21.9 mm
- net OUT3: track 41.6 -> 31.8 mm
- net OUT2: track 36.9 -> 27.0 mm
- net OUT4: track 46.2 -> 36.4 mm
- net Net-(J2-Pin_2): track 6.03 -> 0.00 mm
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Other:
- board text added: "+ -"
- board text added: "BREAD Slice I/O Controller SLC_IOCT R0 11-2025"
- board text removed: "+"
- board text removed: "-"
- board text removed: "BREAD Slice Template SLC_TEMP R3 04-2025"
