File: hardware/BREAD_Slice.kicad_pcb (KiCad board)
At the start: 2 copper layers, 70 x 100 mm, 59 parts, among them J1 Conn_01x10_Socket, J2 Screw_Terminal_01x06, J3 Screw_Terminal_01x02, J4 Screw_Terminal_01x08, SW1 SW_DIP_x04, SW3 SW_SPDT, U1 AP63205, U10 CPC1002N, U11 CPC1002N, U12 NTGS4111PT1G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

Commit message: Added new conenctor
Parts:
- removed J3: Screw_Terminal_01x02, TerminalBlock_Phoenix:TerminalBlock_Phoenix_PT-1,5-2-3.5-H_1x02_P3.50mm_Horizontal
- removed J4: Screw_Terminal_01x08, TerminalBlock_Phoenix:TerminalBlock_Phoenix_PT-1,5-8-3.5-H_1x08_P3.50mm_Horizontal
- J2: value Screw_Terminal_01x06 -> Screw_Terminal_01x16; footprint TerminalBlock_Phoenix:TerminalBlock_Phoenix_PT-1,5-6-3.5-H_1x06_P3.50mm_Horizontal -> kml-custom:1990148
- U12: footprint Package_TO_SOT_SMD:TSOT-23-6 -> Package_SO:TSOP-6_1.65x3.05mm_P0.95mm
- moved R13 23.9 mm to (163.2, 79.7)
- moved R16 23.9 mm to (173.2, 79.6)
- moved U8 23.9 mm to (168.2, 77.6)
- moved R15 22.4 mm to (147.4, 79.7)
- moved R18 22.4 mm to (157.4, 79.6)
- moved U10 22.4 mm to (152.4, 77.6)
- moved R19 20.9 mm to (147.4, 86.8)
- moved R20 20.9 mm to (157.4, 86.8)
- moved U11 20.9 mm to (152.4, 84.8)
- moved J2 20.2 mm to (182.2, 92.9)
- moved U12 18.2 mm to (182.7, 101.5)
- moved D3 18.2 mm to (182.8, 104.7)
- moved R21 18.2 mm to (178.6, 103.2)
- moved SW3 18.2 mm to (173.6, 99.7)
- moved R14 10.2 mm to (163.4, 86.8)
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Connections:
- net OUT1 renamed /OUT1
- net OUT2 renamed /OUT2
- net OUT3 renamed /OUT3
- net OUT4 renamed /OUT4
- J2 pad 1: Net-(J2-Pin_1) -> 24V
- J2 pad 2: Net-(J2-Pin_2) -> GND
- J2 pad 3: Net-(J2-Pin_3) -> OUT4B
- J2 pad 4: IN4B -> /VOUT
- J2 pad 5: IN5B -> OUT3B
- J2 pad 6: IN6B -> /VOUT
- R7 pad 2: Net-(J2-Pin_1) -> Net-(J2-Pin_11)
- R8 pad 2: Net-(J2-Pin_2) -> Net-(J2-Pin_12)
- R9 pad 2: Net-(J2-Pin_3) -> Net-(J2-Pin_13)
- SW3 pad 1: VOUT -> /VOUT
- U12 pad 1: /24V -> 24V
- U12 pad 2: /24V -> 24V
- U12 pad 5: /24V -> 24V
- U12 pad 6: /24V -> 24V
Routing:
- net VOUT: track 69.5 -> 0.00 mm
- net /VOUT: track 0.00 -> 36.2 mm
- net /OUT1: track 32.7 -> 55.6 mm
- net OUT3B: track 8.25 -> 29.8 mm, vias 0 -> 1
- net OUT4B: track 8.26 -> 28.9 mm, vias 0 -> 1
- net +12V: track 124.1 -> 143.7 mm
- net /OUT3: track 41.6 -> 53.0 mm
- net Net-(J2-Pin_12): track 0.00 -> 10.9 mm
- net GND: track 73.4 -> 63.1 mm, vias 35 -> 40
- net Net-(J2-Pin_11): track 0.00 -> 6.66 mm
- net /OUT2: track 36.9 -> 43.4 mm
- net Net-(J2-Pin_2): track 6.03 -> 0.00 mm
- net Net-(J2-Pin_3): track 5.93 -> 0.00 mm
- net Net-(J2-Pin_1): track 5.93 -> 0.00 mm
- net Net-(J2-Pin_13): track 0.00 -> 5.56 mm
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- added copper zone on F.Cu, net 24V
- removed copper zone on F.Cu, net /24V
Other:
- board text added: "BREAD Slice Digital IO SLC_IOCT"
- board text removed: "BREAD Slice Template SLC_TEMP R3 04-2025"

Commit message: updated routing and silkscreen
Parts:
- moved SW3 9.54 mm to (176.8, 108.8), turned to 180 degrees
- moved U12 4.57 mm to (178.2, 101.0)
- moved D3 4.57 mm to (178.3, 104.3)
- moved R21 4.57 mm to (174.1, 102.8)
- moved R10 4.49 mm to (172.5, 62.2)
- moved R12 4.49 mm to (172.5, 55.2)
- moved R2 4.49 mm to (154.8, 68.0)
- moved R3 4.49 mm to (137.8, 61.0)
- moved R4 4.49 mm to (154.8, 60.6)
- moved R6 4.49 mm to (154.8, 54.0)
- moved R7 4.49 mm to (172.5, 72.8)
- moved R8 4.49 mm to (172.5, 69.0)
- moved R9 4.49 mm to (172.5, 65.8)
- moved U2 4.49 mm to (146.0, 68.0)
- moved U3 4.49 mm to (163.0, 68.0)
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Routing:
- net +12V: track 143.7 -> 132.4 mm
- net Net-(D3-K): track 14.5 -> 6.75 mm
- net /VOUT: track 36.2 -> 43.2 mm
- net OUT1B: track 12.7 -> 8.47 mm
- net OUT4B: track 28.9 -> 24.7 mm
- net OUT3B: track 29.8 -> 25.6 mm
- net OUT2B: track 13.4 -> 9.39 mm
- net /IN2: track 74.5 -> 72.7 mm
- net /IN6: track 83.4 -> 81.6 mm
- net /IN4: track 79.3 -> 77.4 mm
- net /OUT1: track 55.6 -> 54.6 mm
- net /IN5: track 81.6 -> 82.2 mm
- net GND: vias 40 -> 41
Other:
- board text added: "IN1"
- board text added: "IN2"
- board text added: "IN3"
- board text added: "IN4"
- board text added: "IN5"
- board text added: "IN6"
- board text removed: "I1"
- board text removed: "I2"
- board text removed: "I3"
- board text removed: "I4"
- board text removed: "I5"
- board text removed: "I6"
