File: hardware/BREAD_Slice.kicad_pcb (KiCad board)
At the start: 2 copper layers, 70 x 100 mm, 55 parts, among them J1 1985195, J2 1990106, J3 1990106, J4 Conn_01x10_Socket, Q1 NTGS4111PT1G, SW1 SW_SPDT, SW2 SW_DIP_x04, SW3 SW_DIP_x04, U1 AP63205, U2 LTV-817S, U3 LTV-817S, U4 LTV-817S, U5 LTV-817S, U6 CPC1002N, U7 CPC1002N, U8 CPC1002N, U9 CPC1002N

Commit message: fix(hw): re-point stale library nicknames
These parts exist in KiCad-Master-Lib; the boards referenced libraries that no
longer exist (kml-custom, KML-Custom, and SparkFun libraries that never
contained the part) or names the library has since changed.

KiCad embeds footprint geometry in the .kicad_pcb, so the boards rendered and
fabricated correctly and the rot stayed invisible -- it only surfaces on
update-from-library, or when a generator tries to resolve a nickname.

Nickname/name only. No geometry is changed:

  KMLib_Mounting:Thermal Pad -> KMLib_Mounting:Thermal_Pad
  kml-custom:FAST-Logo-Medium -> KMLib_Aesthetic:FAST-Logo-Medium
  kml-custom:OSHW_Logo_8mm -> KMLib_Aesthetic:OSHW_Logo_8mm

Only references that failed to resolve were touched. Generic parts (<=4 pins)
and KiCad *-rescue libraries are deliberately excluded: fingerprint matching
cannot distinguish a 2-pin resistor from a 2-pin capacitor, so those are being
done by hand.
Parts:
- G***: footprint kml-custom:FAST-Logo-Medium -> KMLib_Aesthetic:FAST-Logo-Medium
- HS1: footprint KMLib_Mounting:Thermal Pad -> KMLib_Mounting:Thermal_Pad
- Ref**: footprint kml-custom:OSHW_Logo_8mm -> KMLib_Aesthetic:OSHW_Logo_8mm
Changed lines of the file:
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@@
 		)
 	)
-	(footprint "kml-custom:OSHW_Logo_8mm"
+	(footprint "KMLib_Aesthetic:OSHW_Logo_8mm"
 		(layer "F.Cu")
 		(at 135.950001 107.8 -90)
@@
 		)
 	)
-	(footprint "kml-custom:FAST-Logo-Medium"
+	(footprint "KMLib_Aesthetic:FAST-Logo-Medium"
 		(layer "F.Cu")
 		(at 130.1 70.3 -90)
@@
 		)
 	)
-	(footprint "KMLib_Mounting:Thermal Pad"
+	(footprint "KMLib_Mounting:Thermal_Pad"
 		(layer "F.Cu")
 		(at 131.8 121.45)
