File: hardware/slice_template.kicad_sch (KiCad schematic)
At the start: 19 parts, among them J1 Conn_01x10_Socket, SW1 SW_DIP_x04, U1 AP63205

Commit message: finalize revision of schematic
Parts:
- renumbered J1 to J4, SW1 to SW2
Changed lines of the file:
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@@
 		(on_board yes)
 		(dnp no)
-		(property "Reference" "SW1"
+		(property "Reference" "SW2"
 			(at 165.1 82.804 0)
 			(effects
@@
 			(project "BREAD_Slice"
 				(path "/66043bca-a260-4915-9fce-8a51d324c687/a4d66d05-b498-454f-8d54-68b671c284b9"
-					(reference "SW1")
+					(reference "SW2")
 					(unit 1)
 				)
@@
 		(on_board yes)
 		(dnp no)
-		(property "Reference" "J1"
+		(property "Reference" "J4"
 			(at 24.892 85.852 0)
 			(effects
@@
 			(project ""
 				(path "/66043bca-a260-4915-9fce-8a51d324c687/a4d66d05-b498-454f-8d54-68b671c284b9"
-					(reference "J1")
-					(unit 1)
-				)
+					(reference "J4")
+					(unit 1)
+				)

Commit message: revision of symbol attachment and clear out old layout and start new; kml-custom to kmlib-local
Parts:
- A1: footprint kml-custom:Arduino_Nano_Headers -> KMLib_Boards_Modules:Arduino_Nano_Headers
- D2: footprint kml-custom:WS2812-5050-4PIN -> KMLib_IC_SMD:WS2812-5050-4PIN
- HS1: footprint kml-custom:Thermal Pad -> KMLib_Mounting:Thermal Pad
- U1: footprint kml-custom:SOIC_05WU-7_DIO-M -> KMLib_IC_SMD:SOIC_05WU-7_DIO
Changed lines of the file:
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@@
 			)
 		)
-		(property "Footprint" "kml-custom:Arduino_Nano_Headers"
+		(property "Footprint" "KMLib_Boards_Modules:Arduino_Nano_Headers"
 			(at 237.49 81.28 0)
 			(effects
@@
 			)
 		)
-		(property "Footprint" "kml-custom:SOIC_05WU-7_DIO-M"
+		(property "Footprint" "KMLib_IC_SMD:SOIC_05WU-7_DIO"
 			(at 113.03 93.98 0)
 			(effects
@@
 			)
 		)
-		(property "Footprint" "kml-custom:WS2812-5050-4PIN"
+		(property "Footprint" "KMLib_IC_SMD:WS2812-5050-4PIN"
 			(at 190.5 142.24 0)
 			(effects
@@
 			)
 		)
-		(property "Footprint" "kml-custom:Thermal Pad"
+		(property "Footprint" "KMLib_Mounting:Thermal Pad"
 			(at 68.2752 107.95 0)
 			(effects

Commit message: update all to KMLib, untrack backups in gitignore, and revise routing on board to simplify
Parts:
- A1: footprint KMLib_Boards_Modules:Arduino_Nano_Headers -> KMLib_Boards_Modules:Arduino_Nano; symbol kml-custom:Arduino_Nano_v3.x -> KMLib_IC_MCU_MPU:Arduino_Nano_v3.x
- D1: footprint Diode_SMD:D_SOD-123F -> Diode_THT:D_DO-41_SOD81_P10.16mm_Horizontal
- D2: symbol kml-custom:WS2812B_5050 -> KMLib_IC_Digital:WS2812B_5050_RGB_LED
- U1: symbol kml-custom:AP63205WU-7 -> KMLib_IC_Power:AP63205WU-7_Buck_Regulator
Changed lines of the file:
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@@
 			)
 		)
-		(property "Description" ""
+		(property "Description" "Mounting Hole without connection"
 			(at 110.49 133.35 0)
 			(effects
@@
 			)
 		)
-		(property "Description" ""
+		(property "Description" "Mounting Hole without connection"
 			(at 110.49 143.51 0)
 			(effects
@@
 			)
 		)
-		(property "Description" ""
+		(property "Description" "Mounting Hole without connection"
 			(at 125.73 133.35 0)
 			(effects
@@
 			)
 		)
-		(property "Description" ""
+		(property "Description" "Mounting Hole without connection"
 			(at 125.73 143.51 0)
 			(effects
@@
 	)
 	(symbol
-		(lib_id "kml-custom:Arduino_Nano_v3.x")
+		(lib_id "KMLib_IC_MCU_MPU:Arduino_Nano_v3.x")
 		(at 237.49 81.28 0)
 		(unit 1)
@@
 			)
 		)
-		(property "Footprint" "KMLib_Boards_Modules:Arduino_Nano_Headers"
+		(property "Footprint" "KMLib_Boards_Modules:Arduino_Nano"
 			(at 237.49 81.28 0)
 			(effects
@@
 			)
 		)
-		(property "Description" ""
+		(property "Description" "Unpolarized capacitor, small symbol"
 			(at 129.54 92.71 0)
 			(effects
@@
 			)
 		)
-		(property "Description" ""
+		(property "Description" "Unpolarized capacitor, small symbol"
 			(at 129.54 102.87 0)
 			(effects
@@
 	)
 	(symbol
-		(lib_id "kml-custom:AP63205WU-7")
+		(lib_id "KMLib_IC_Power:AP63205WU-7_Buck_Regulator")
 		(at 113.03 93.98 0)
 		(unit 1)
@@
 	)
 	(symbol
-		(lib_id "kml-custom:WS2812B_5050")
+		(lib_id "KMLib_IC_Digital:WS2812B_5050_RGB_LED")
 		(at 173.99 133.35 0)
 		(mirror y)
@@
 			)
 		)
-		(property "Footprint" "Diode_SMD:D_SOD-123F"
+		(property "Footprint" "Diode_THT:D_DO-41_SOD81_P10.16mm_Horizontal"
 			(at 160.02 43.815 0)
 			(effects
@@
 			)
 		)
-		(property "Description" ""
+		(property "Description" "Inductor, small symbol"
 			(at 129.54 97.79 0)
 			(effects
@@
 			)
 		)
-		(property "Description" ""
+		(property "Description" "Unpolarized capacitor, small symbol"
 			(at 139.7 102.87 0)
 			(effects
@@
 			)
 		)
-		(property "Description" ""
+		(property "Description" "Unpolarized capacitor, small symbol"
 			(at 95.25 102.87 0)
 			(effects

Commit message: added dip switches to IOCT
Changed lines of the file:
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@@
+	(wire
+		(pts
+			(xy 254 142.24) (xy 267.97 142.24)
+		)
+		(stroke
+			(width 0)
+			(type default)
+			(color 0 194 0 1)
+		)
+	)
 	(wire
 		(pts
@@
 		)
 	)
+	(label "ESTOP"
+		(at 254 142.24 0)
+		(effects
+			(font
+				(size 1.27 1.27)
+			)
+			(justify left bottom)
+		)
+	)
 	(label "LED"
 		(at 187.96 133.35 180)
@@
 		(effects
 			(font
+				(size 1.27 1.27)
+			)
+			(justify left)
+		)
+	)
+	(hierarchical_label "ESTOP"
+		(shape input)
+		(at 267.97 142.24 0)
+		(effects
+			(font
